File: Hardware/Body_PCB_v1.sch (EAGLE design)
At the start: 0 parts

Commit message: Addition of 2D Vertical Surface Code
- Added code for Vertical Steps
- No feedback from Z Axis motors
- Andrew. This is for you.
Parts:
- added C1, C2, C3, C4: (no value), Team_Ojas_OVPowar:C1206
- added JP1, JP13, JP2, JP3, JP4: (no value), SparkFun-Connectors:M04PTH
- added JP10, JP11, JP9: FEMALE 2x3, SparkFun-Connectors:M03X2FEMALE
- added JP5, JP6: (no value), SparkFun-Connectors:M03PTH
- added JP7, JP8: (no value), SparkFun-Connectors:M05PTH
- added R1, R11, R13, R15, R3, R5, R7, R9: 1kOhm, Team_Ojas_OVPowar:R0805
- added R10, R12, R14, R16, R2, R4, R6, R8: 2kOhm, Team_Ojas_OVPowar:R0805
- added SJ1, SJ2: (no value), jumper:SJ2W
- added U$1, U$2: TB6612FNG, Team_Ojas_OVPowar:TB6612FNG
- added U$3, U$4: MOLEX-SMT-2-PIN-VERTICAL, Team_Ojas_OVPowar:MOLEX-SMT-2-PIN-VERTICAL
- added U1: MBED_NXP_LPC1768, Team_Ojas_OVPowar:MBED_NXP_LPC1768
- added U2: 1117, Carnot_AfterMarket_v2.2:1117
Connections:
- new net 12VIN: C2.1, JP11.1, JP11.2, U$1.VM, U$2.VM
- new net 3.3V: C4.1, JP13.4, JP7.5, JP8.5, U$1.STANDBY, U$2.STANDBY, U2.VOUT
- new net 5VIN: C1.1, C3.1, JP1.1, JP10.6, JP11.3, JP11.4, JP2.1, JP3.1, JP4.1, JP5.1, JP6.1, JP9.6, U$1.VCC, U$2.VCC, U1.VIN, U2.VIN
- new net EXTRA1: SJ1.2, U1.P14/RX
- new net EXTRA2: SJ2.2, U1.P18/A3
- new net EXTRA_ANALOG1: U1.P19/A4
- new net EXTRA_ANALOG2: U1.P20/A5
- new net GND: C1.2, C2.2, C3.2, C4.2, JP1.4, JP10.5, JP11.5, JP11.6, JP13.1, JP2.4, JP3.4, JP4.4, JP5.3, JP6.3, JP7.1, JP8.1, JP9.5, R10.1, R12.1, R14.1, R16.1, R2.1, R4.1, R6.1, R8.1, U$1.GND, U$2.GND, U$3.2, U$4.2, U1.GND, U2.GND
- new net PRESSURE_SENSOR: U1.P17/A2
- new net SERVO1: JP5.2, SJ1.3
- new net SERVO2: JP6.2, SJ2.3
- new net SOLENOID1: JP13.2, U$3.1, U1.P27/SCL/RX
- new net SOLENOID2: JP13.3, U$4.1, U1.P28/SDA/TX
- new net ULTRASONIC_BOTTOM_ECHO: R7.1, R8.2, U1.P8
- new net ULTRASONIC_BOTTOM_ECHO_5V: JP4.3, R7.2
- new net ULTRASONIC_LEFT_ECHO: R1.1, R2.2, U1.P5/MOSI
- new net ULTRASONIC_LEFT_ECHO_5V: JP1.3, R1.2
- new net ULTRASONIC_RIGHT_ECHO: R5.1, R6.2, U1.P7/SCK
- new net ULTRASONIC_RIGHT_ECHO_5V: JP3.3, R5.2
- new net ULTRASONIC_TOP_ECHO: R3.1, R4.2, U1.P6/MISO
- new net ULTRASONIC_TOP_ECHO_5V: JP2.3, R3.2
- new net ULTRASONIC_TRIGGER: JP1.2, JP2.2, JP3.2, JP4.2, U1.P11/MOSI
- new net X+: JP7.3, U$1.A01
- new net X-: JP7.4, U$1.A02
- new net X_AXIS_DOWN: U$1.AI2, U1.P12/MISO
- new net X_AXIS_SPEED: U$1.PWMA, U1.P21/PWM0
- new net X_AXIS_UP: U$1.AI1, U1.P9/SDA/TX
- new net X_POS: JP7.2, U1.P15/A0
- new net Y+: JP8.3, U$1.B02
- new net Y-: JP8.4, U$1.B01
- new net Y_AXIS_DOWN: U$1.BI2, U1.P13/SCK/TX
- new net Y_AXIS_SPEED: U$1.PWMB, U1.P22/PWM1
- new net Y_AXIS_UP: U$1.BI1, U1.P10/SCL/RX
- new net Y_POS: JP8.2, U1.P16/A1
- new net Z1+: JP9.2, U$2.A01
- new net Z1-: JP9.4, U$2.A02
- new net Z1_POS+: R10.2, R9.1, U1.P30/CANRX
- new net Z1_POS+_5V: JP10.3, R9.2
- new net Z1_POS-: R13.1, R14.2, SJ1.1
- new net Z1_POS-_5V: JP10.1, R13.2
- new net Z2+: JP10.2, U$2.B02
- new net Z2-: JP10.4, U$2.B01
- new net Z2_POS+: R11.1, R12.2, U1.P29/CANTX
- new net Z2_POS+_5V: JP9.3, R11.2
- new net Z2_POS-: R15.1, R16.2, SJ2.1
- new net Z2_POS-_5V: JP9.1, R15.2
- new net Z_AXIS1_SPEED: U$2.PWMA, U1.P23/PWM2
- new net Z_AXIS2_SPEED: U$2.PWMB, U1.P24/PWM3
- new net Z_AXIS_DOWN: U$2.AI2, U$2.BI2, U1.P26/PWM5
- new net Z_AXIS_UP: U$2.AI1, U$2.BI1, U1.P25/PWM4
Other:
- note added: "LIMIT SWITCH via DIODE Jumper for Servo 1 and 2 Jumper for LIS3DH Jumper shifts Direction to NAND Gate"
- note added: "NXP LPC1768 5V/12V to 3.3V Voltage Dividers 3.3V to 5V/12V Level Shifters Power Regulators"
- note added: "Solenoid 1,2 Actuator 1,2 DC Motor 1,2,3,4"
- note added: "Ultrasonic 1,2,3,4"
- note removed: "12V-5V Regulator"
- note removed: "5V-3.3V Regulator"
- note removed: "Air Filter Clog"
- note removed: "Battery Charge"
- note removed: "Battery_Voltage"
- note removed: "DOC"
- note removed: "EXTERNAL GPS"
- note removed: "FUEL_GAUGE"
- note removed: "High Beam"
- note removed: "Ignition"
- note removed: "Illumination"
- note removed: "Input Protection Circuit"
- note removed: "MAGNETOMETER"
- note removed: "Neutral"
- note removed: "OBD_CAR"
- note removed: "Oil Pressure"
- note removed: "Park Brake"
- note removed: "RPM"
- note removed: "RPM using Current Sensor"
- note removed: "Temperature Sensor"
- note removed: "Throttle"
- note removed: "Turn Left"
- note removed: "Turn Right"
